File: 14000JKFF.kicad_pcb (KiCad board)
At the start: 2 copper layers, 96.3 x 94.8 mm, 122 parts, among them IC1 74LVC1G3157DW-7, IC10 NE555DR, IC11 SN74AHC1G04DBVR, IC12 SN74AHC1G04DBVR, IC13 SN74AHC1G04DBVR, IC14 74AHC573PW,118, IC15 74AHC574D,118, IC16 74AHC574D,118, IC2 74AHC573PW,118, IC20 SN74AHC1G02DBVR, IC21 SN74AHC1G02DBVR, IC23 74AHC00D,118, IC24 74AHC32D,118, IC25 74AHC74PW,118, IC26 74AHC74PW,118, IC28 74AHC1G79GW,125, IC29 74HC04D_BJ_, IC3 74LVC1G3157DW-7, IC30 74AHC1G79GW,125, IC33 NE555DR, IC34 74HC04D_BJ_, IC35 SN74AHC1G04DBVR, IC4 74LVC1G3157DW-7, IC5 74LVC1G3157DW-7, IC6 74LVC1G3157DW-7, J2 USB4125-GF-A, SW1 SW_Push, SW2 SW_Push, SW3 SW_Push, SW4 SW_DIP_x05, SW5 SW_DIP_x07, SW8 SW_DIP_x05, SW9 SW_DIP_x05, U1 SN74AHC1G08DBVR, U2 SN74AHC1G08DBVR, X1 4K7, X2 10K

Commit message: 14000JKFF 1.1.0
Parts:
- removed C15, C26: 100nF, Capacitor_SMD:C_1206_3216Metric
- removed IC14: 74AHC573PW,118, AAAAAAAAA:SOIC127P1032X265-20N
- removed IC25: 74AHC74PW,118, AAAAAAAAA:SOP65P640X110-14N
- added C2: 100nF, Capacitor_SMD:C_1206_3216Metric, F.Cu at (165.0, 121.9)
- added IC7: 74AHC573PW,118, AAAAAAAAA:SOP65P640X110-20N, F.Cu at (163.5, 126.8)
- IC2: footprint AAAAAAAAA:SOIC127P1032X265-20N -> AAAAAAAAA:SOP65P640X110-20N
- moved C3 2.94 mm to (161.7, 115.0)
- moved IC2 2.09 mm to (163.2, 110.2)
Connections:
- IC15 pad 4: unconnected-(IC15-D2-Pad4) -> GND
- IC15 pad 5: unconnected-(IC15-D3-Pad5) -> GND
- IC15 pad 6: unconnected-(IC15-D4-Pad6) -> GND
- IC15 pad 7: unconnected-(IC15-D5-Pad7) -> GND
- IC15 pad 8: unconnected-(IC15-D6-Pad8) -> GND
- IC15 pad 9: unconnected-(IC15-D7-Pad9) -> GND
- IC16 pad 4: unconnected-(IC16-D2-Pad4) -> GND
- IC16 pad 5: unconnected-(IC16-D3-Pad5) -> GND
- IC16 pad 6: unconnected-(IC16-D4-Pad6) -> GND
- IC16 pad 7: unconnected-(IC16-D5-Pad7) -> GND
- IC16 pad 8: unconnected-(IC16-D6-Pad8) -> GND
- IC16 pad 9: unconnected-(IC16-D7-Pad9) -> GND
- IC2 pad 3: unconnected-(IC2-D1-Pad3) -> GND
- IC2 pad 4: unconnected-(IC2-D2-Pad4) -> GND
- IC2 pad 5: unconnected-(IC2-D3-Pad5) -> GND
- IC2 pad 6: unconnected-(IC2-D4-Pad6) -> GND
- IC2 pad 7: unconnected-(IC2-D5-Pad7) -> GND
- IC2 pad 8: unconnected-(IC2-D6-Pad8) -> GND
- IC2 pad 9: unconnected-(IC2-D7-Pad9) -> GND
- IC24 pad 12: unconnected-(IC24-4A-Pad12) -> GND
- IC24 pad 13: unconnected-(IC24-4B-Pad13) -> GND
- IC26 pad 11: unconnected-(IC26-2CP-Pad11) -> Net-(IC24-1Y)
- IC26 pad 12: unconnected-(IC26-2D-Pad12) -> /First toggle/JANDK
- IC26 pad 13: unconnected-(IC26-2~{RD}-Pad13) -> /First toggle/JANDK
- IC26 pad 9: unconnected-(IC26-2Q-Pad9) -> /First toggle/TNE
- IC29 pad 11: unconnected-(IC29-5A-Pad11) -> GND
- IC29 pad 13: unconnected-(IC29-6A-Pad13) -> GND
- IC29 pad 3: unconnected-(IC29-2A-Pad3) -> GND
- IC29 pad 5: unconnected-(IC29-3A-Pad5) -> GND
- IC34 pad 11: unconnected-(IC34-5A-Pad11) -> GND
- IC34 pad 13: unconnected-(IC34-6A-Pad13) -> GND
Routing:
- net +5V: track 550.1 -> 527.2 mm, vias 27 -> 26
- net /First toggle/TNE: track 45.5 -> 57.5 mm, vias 3 -> 5
- net Net-(IC24-1Y): track 12.2 -> 21.5 mm, vias 2 -> 0
- net GND: track 25.3 -> 30.0 mm, vias 186 -> 251
- net /First toggle/JANDK: track 153.1 -> 157.4 mm
- net /Klopení vstupů/KLATCHED: track 35.8 -> 32.7 mm
- net /Klopení vstupů/JLATCHED: track 44.5 -> 41.6 mm
- net /First toggle/NOTJANDK: track 193.3 -> 191.2 mm
- net /First toggle/CLK: track 192.2 -> 190.6 mm
- net /SR LATCH/SRLATCH: track 112.9 -> 114.5 mm
- net Net-(IC2-Q0): track 114.7 -> 113.2 mm
- net /toggling/TOG4: track 53.8 -> 54.6 mm
Other:
- board text added: "14000 JK FFs 1.1.0"
- board text removed: "14000 JK FFs 1.0.0"

Commit message: Add files via upload
Parts:
- moved D6 2.60 mm to (117.8, 115.5)
- moved R11 2.50 mm to (117.8, 118.0)
- moved D7 2.50 mm to (117.0, 87.9)
- moved R12 2.30 mm to (117.0, 90.3)
Connections:
- IC6 pad 1: Net-(IC3-B1) -> /toggling/TOGGLE
- IC6 pad 3: /First toggle/FT -> Net-(IC2-Q0)
- IC6 pad 4: /toggling/TOGGLE -> Net-(IC3-B1)
- IC6 pad 6: Net-(IC2-Q0) -> /First toggle/FT
Routing:
- net GND: track 30.0 -> 35.0 mm, vias 251 -> 255
- net /First toggle/FT: track 74.8 -> 79.5 mm
- net Net-(IC3-B1): track 10.9 -> 6.61 mm
- net /toggling/TOGGLE: track 38.7 -> 42.8 mm
- net +5V: track 527.2 -> 529.4 mm
- net Net-(IC2-Q0): track 113.2 -> 111.9 mm, vias 2 -> 3
Other:
- board text added: "14000 JK FFs 1.2.0"
- board text removed: "14000 JK FFs 1.1.0"

Commit message: version 1.3
Parts:
- removed C41: 100nF, Capacitor_SMD:C_1206_3216Metric
- added C15: 100nF, Capacitor_SMD:C_1206_3216Metric, F.Cu at (94.0, 86.3)
- added J1: Conn_01x01, Connector_PinHeader_2.54mm:PinHeader_1x01_P2.54mm_Vertical, F.Cu at (118.7, 162.6)
- added J3: Conn_01x01, Connector_PinHeader_2.54mm:PinHeader_1x01_P2.54mm_Vertical, F.Cu at (142.2, 155.8)
- added J4: Conn_01x01, Connector_PinHeader_2.54mm:PinHeader_1x01_P2.54mm_Vertical, F.Cu at (160.4, 155.7)
- added J5: Conn_01x01, Connector_PinHeader_2.54mm:PinHeader_1x01_P2.54mm_Vertical, F.Cu at (113.0, 73.6)
- moved D4 2.52 mm to (161.2, 139.4)
- moved R7 2.50 mm to (99.4, 142.3)
- moved D3 2.50 mm to (141.5, 139.5)
- moved R5 2.40 mm to (141.5, 142.1)
- moved D5 2.40 mm to (99.4, 139.8)
- moved R6 2.32 mm to (161.2, 141.9)
- moved S2 0.30 mm to (160.4, 148.2)
- moved S1 0.15 mm to (142.2, 148.3)
Connections:
- IC26 pad 10: unconnected-(IC26-2~{SD}-Pad10) -> +5V
- IC26 pad 4: unconnected-(IC26-1~{SD}-Pad4) -> +5V
- IC6 pad 2: +5V -> GND
- IC6 pad 5: GND -> +5V
Routing:
- net Net-(D1-A): track 20.9 -> 30.6 mm
- net +5V: track 529.4 -> 535.2 mm, vias 26 -> 27
- net /Vstupy/Tlačítko1/TLA: track 52.1 -> 57.7 mm
- net /Vstupy/Tlačítko/TLA: track 22.5 -> 28.0 mm
- net /toggling/TOGGLE: track 42.8 -> 37.5 mm
- net /First toggle/FT: track 79.5 -> 75.2 mm
- net Net-(IC34-4A): track 48.5 -> 51.8 mm
- net /Klopení vstupů/J: track 108.0 -> 110.6 mm
- net /First toggle/CLK: track 190.6 -> 193.0 mm
- net /Klopení vstupů/K: track 116.3 -> 118.4 mm
- net Net-(IC34-2Y): track 53.2 -> 54.4 mm
- net GND: track 35.0 -> 35.7 mm, vias 255 -> 261
Other:
- board text added: "14000 JK FFs 1.3.0"
- board text added: "EXT J"
- board text added: "EXT K"
- board text added: "EXT OUT"
- board text added: "EXT. CL."
- board text removed: "14000 JK FFs 1.2.0"
