File: firstToggle.kicad_sch (KiCad schematic)
At the start: 17 parts, among them IC23 74AHC00D,118, IC24 74AHC32D,118, IC25 74AHC74PW,118, IC26 74AHC74PW,118, IC5 74LVC1G3157DW-7, SW4 SW_DIP_x05, U2 SN74AHC1G08DBVR

Commit message: 14000JKFF 1.1.0
Parts:
- removed C26: 100nF, Capacitor_SMD:C_1206_3216Metric, symbol Device:C
- removed IC25: 74AHC74PW,118, AAAAAAAAA:SOP65P640X110-14N, symbol AAAAAAAAAA:74AHC74PW,118
Connections:
- net GND: now also IC24.12 (4A), IC24.13 (4B)
- net JANDK: now also IC26.12 (2D), IC26.13 (2~{RD})
- net TNE: now also IC26.9 (2Q)
- net at IC24.3 (1Y): now also IC26.11 (2CP)
- no-connect marks 19 -> 5
Other:
- note removed: "D (NE) S PRESETEM A CLEAREM"

Commit message: version 1.3
Connections:
- net +5V: now also IC26.10 (2~{SD}), IC26.4 (1~{SD})
- no-connect marks 5 -> 3
Changed lines of the file:
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@@
-	)
-	(no_connect
-		(at 180.34 49.53)
-	)
-	(no_connect
-		(at 152.4 46.99)
 	)
 	(no_connect
@@
 	)
 	(symbol
+		(lib_id "power:+5V")
+		(at 180.34 49.53 270)
+		(unit 1)
+		(exclude_from_sim no)
+		(in_bom yes)
+		(on_board yes)
+		(dnp no)
+		(property "Reference" "#PWR0153"
+			(at 176.53 49.53 0)
+			(effects
+				(font
+					(size 1.27 1.27)
+				)
+				(hide yes)
+			)
+		)
+		(property "Value" "+5V"
+			(at 184.15 49.53 0)
+			(effects
+				(font
+					(size 1.27 1.27)
+				)
+			)
+		)
+		(property "Footprint" ""
+			(at 180.34 49.53 0)
+			(effects
+				(font
+					(size 1.27 1.27)
+				)
+				(hide yes)
+			)
+		)
+		(property "Datasheet" ""
+			(at 180.34 49.53 0)
+			(effects
+				(font
+					(size 1.27 1.27)
+				)
+				(hide yes)
+			)
+		)
+		(property "Description" ""
+			(at 180.34 49.53 0)
+			(effects
+				(font
+					(size 1.27 1.27)
+				)
+				(hide yes)
+			)
+		)
+		(pin "1"
+		)
+		(instances
+			(project "14000JKFF"
+				(path "/56463b8e-670e-41df-bd3a-314161dc4bc4/df53b169-e5a4-412e-9dd1-7763e315ffc5"
+					(reference "#PWR0153")
+					(unit 1)
+				)
+			)
+		)
+	)
+	(symbol
 		(lib_id "AAAAAAAAAA:74AHC32D,118")
 		(at 93.98 41.91 0)
@@
 					(unit 1)
 				)
+			)
+		)
+	)
+	(symbol
+		(lib_id "power:+5V")
+		(at 152.4 46.99 90)
+		(unit 1)
+		(exclude_from_sim no)
+		(in_bom yes)
+		(on_board yes)
+		(dnp no)
+		(property "Reference" "#PWR0152"
+			(at 156.21 46.99 0)
+			(effects
+				(font
+					(size 1.27 1.27)
+				)
+				(hide yes)
+			)
+		)
+		(property "Value" "+5V"
+			(at 148.59 46.99 0)
+			(effects
+				(font
+					(size 1.27 1.27)
+				)
+			)
+		)
+		(property "Footprint" ""
+			(at 152.4 46.99 0)
+			(effects
+				(font
+					(size 1.27 1.27)
+				)
+				(hide yes)
+			)
+		)
+		(property "Datasheet" ""
+			(at 152.4 46.99 0)
+			(effects
+				(font
+					(size 1.27 1.27)
+				)
+				(hide yes)
+			)
+		)
+		(property "Description" ""
+			(at 152.4 46.99 0)
+			(effects
+				(font
+					(size 1.27 1.27)
+				)
+				(hide yes)
+			)
+		)
+		(pin "1"
+		)
+		(instances
+			(project "14000JKFF"
+				(path "/56463b8e-670e-41df-bd3a-314161dc4bc4/df53b169-e5a4-412e-9dd1-7763e315ffc5"
+					(reference "#PWR0152")
+					(unit 1)
+				)
