File: klopeni_vstupu.kicad_sch (KiCad schematic)
At the start: 12 parts, among them IC1 74LVC1G3157DW-7, IC14 74AHC573PW,118, IC15 74AHC574D,118, IC16 74AHC574D,118, IC4 74LVC1G3157DW-7, SW8 SW_DIP_x05, SW9 SW_DIP_x05

Commit message: 14000JKFF 1.1.0
Parts:
- removed C15: 100nF, Capacitor_SMD:C_1206_3216Metric, symbol Device:C
- removed IC14: 74AHC573PW,118, AAAAAAAAA:SOIC127P1032X265-20N, symbol AAAAAAAAAA:74AHC573PW,118
- added C2: 100nF, Capacitor_SMD:C_1206_3216Metric, symbol Device:C
- added IC7: 74AHC573PW,118, AAAAAAAAA:SOP65P640X110-20N, symbol AAAAAAAAAA:74AHC573PW,118
Connections:
- net +5V: now also C2.2, IC7.20 (VCC)
- net CLK: now also IC7.11 (LE)
- net GND: now also IC15.4 (D2), IC15.5 (D3), IC15.6 (D4), IC15.7 (D5), IC15.8 (D6), IC15.9 (D7), IC16.4 (D2), IC16.5 (D3), IC16.6 (D4), IC16.7 (D5), IC16.8 (D6), IC16.9 (D7), C2.1, IC7.1 (~{OE}), IC7.10 (GND), IC7.4 (D2), IC7.5 (D3), IC7.6 (D4), IC7.7 (D5), IC7.8 (D6), IC7.9 (D7)
- net J: now also IC7.2 (D0)
- net JLATCHED: now also IC7.19 (Q0)
- net K: now also IC7.3 (D1)
- net KLATCHED: now also IC7.18 (Q1)
- no-connect marks 36 -> 18
Other:
- note added: "D LATCH"
- note removed: "D LATCH transparentní"
