File: napajeni.kicad_sch (KiCad schematic)
At the start: 6 parts, among them J2 USB4125-GF-A

Commit message: 14000JKFF 1.1.0
Connections:
- no-connect marks 0 -> 4
Changed lines of the file:
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@@
 		(color 0 0 0 0)
+	)
+	(no_connect
+		(at 30.48 100.33)
+	)
+	(no_connect
+		(at 30.48 97.79)
+	)
+	(no_connect
+		(at 30.48 95.25)
+	)
+	(no_connect
+		(at 30.48 102.87)
 	)
 	(wire
