File: toggling.kicad_sch (KiCad schematic)
At the start: 15 parts, among them IC28 74AHC1G79GW,125, IC29 74HC04D_BJ_, IC30 74AHC1G79GW,125, IC33 NE555DR, SW5 SW_DIP_x07

Commit message: 14000JKFF 1.1.0
Connections:
- net GND: now also IC29.11 (5A), IC29.13 (6A), IC29.3 (2A), IC29.5 (3A)
- no-connect marks 8 -> 4
